Commit message: Base Ready

File: src/robot_description/urdf/robot_base.urdf.xacro (robot description, xacro)
@@ -1,6 +1,12 @@
 <?xml version="1.0" ?>
 <robot xmlns:xacro="http://ros.org/wiki/xacro" name="robot_base">
-    <xacro:include filename="robot_essentials.xacro" />
+    <xacro:include filename="$(find robot_description)/urdf/robot_essentials.xacro" />
+    <xacro:include filename="$(find robot_description)/urdf/gazebo_essentials_base.xacro" />
     <link name="base_link">
+        <inertial>
+            <origin xyz="0.0030946 4.78250032638821E-11 0.053305" rpy="0 0 0" />
+            <mass value="47.873" />
+            <inertia ixx="0.774276574699151" ixy="-1.03781944357671E-10" ixz="0.00763014265820928" iyy="1.64933255189991" iyz="1.09578155845563E-12" izz="2.1239326987473" />
+        </inertial>
         <visual>
             <origin xyz="0 0 0" rpy="1.5707963267949 0 3.14" />
@@ -12,4 +18,10 @@
             </material>
         </visual>
+        <collision>
+            <origin xyz="0 0 0" rpy="1.5707963267949 0 3.14" />
+            <geometry>
+                <mesh filename="package://robot_description/meshes/robot_base.stl" />
+            </geometry>
+        </collision>
     </link>
     <xacro:robot_wheel prefix="rear_left" />
@@ -21,3 +33,11 @@
     <xacro:wheel_joint prefix="rear_left" origin="-0.220 0.250 0" />
     <xacro:wheel_joint prefix="rear_right" origin="-0.220 -0.250 0" />
+    <xacro:base_transmission prefix="front_left" />
+    <xacro:base_transmission prefix="front_right" />
+    <xacro:base_transmission prefix="rear_left" />
+    <xacro:base_transmission prefix="rear_right" />
+    <xacro:wheel_friction prefix="front_left" />
+    <xacro:wheel_friction prefix="front_right" />
+    <xacro:wheel_friction prefix="rear_left" />
+    <xacro:wheel_friction prefix="rear_right" />
 </robot>

File: src/robot_description/urdf/robot_essentials.xacro (robot description, xacro)
@@ -3,4 +3,9 @@
     <xacro:macro name="robot_wheel" params="prefix">
         <link name="${prefix}_wheel">
+            <inertial>
+                <origin xyz="-4.1867E-18 0.0068085 -1.65658661799998E-18" rpy="0 0 0" />
+                <mass value="2.6578" />
+                <inertia ixx="0.00856502765719703" ixy="1.5074118157338E-19" ixz="-4.78150098725052E-19" iyy="0.013670640432096" iyz="-2.68136447099727E-19" izz="0.00856502765719703" />
+            </inertial>
             <visual>
                 <origin xyz="0 0 0" rpy="1.5707963267949 0 0" />
@@ -12,8 +17,14 @@
                 </material>
             </visual>
+            <collision>
+                <origin xyz="0 0 0" rpy="1.5707963267949 0 0" />
+                <geometry>
+                    <mesh filename="package://robot_description/meshes/wheel.stl" />
+                </geometry>
+            </collision>
         </link>
     </xacro:macro>
     <xacro:macro name="wheel_joint" params="prefix origin">
-        <joint name="${prefix}_wheel_joint" type="fixed">
+        <joint name="${prefix}_wheel_joint" type="continuous">
             <axis xyz="0 1 0" />
             <parent link="base_link" />
@@ -22,3 +33,15 @@
         </joint>
     </xacro:macro>
+    <xacro:macro name="base_transmission" params="prefix ">
+        <transmission name="${prefix}_wheel_trans" type="SimpleTransmission">
+            <type>transmission_interface/SimpleTransmission</type>
+            <actuator name="${prefix}_wheel_motor">
+                <hardwareInterface>hardware_interface/VelocityJointInterface</hardwareInterface>
+                <mechanicalReduction>1</mechanicalReduction>
+            </actuator>
+            <joint name="${prefix}_wheel_joint">
+                <hardwareInterface>hardware_interface/VelocityJointInterface</hardwareInterface>
+            </joint>
+        </transmission>
+    </xacro:macro>
 </robot>
