Commit message: mobile_manipulator.urdf working but code developed by me is not

File: src/robot_description/urdf/robot_arm.urdf.xacro (robot description, xacro)
@@ -3,5 +3,5 @@
     <xacro:include filename="$(find robot_description)/urdf/robot_arm_essentials.xacro" />
     <xacro:include filename="$(find robot_description)/urdf/gazebo_essentials_arm.xacro" />
-    <link name="world"/>
+    <link name="base_link"></link>
     <link name="arm_base">
         <inertial>
@@ -114,5 +114,5 @@
         </collision>
     </link>
-    <xacro:arm_joint prefix="arm_base" parent="world" child="arm_base" originxyz="0.0 0.0 0.1" originrpy="0 0 0"/>
+    <xacro:arm_joint prefix="arm_base" parent="base_link" child="arm_base" originxyz="0.0 0.0 0.1" originrpy="0 0 0"/>
     <xacro:arm_joint prefix="shoulder" parent="arm_base" child="bicep" originxyz="-0.05166 0.0 0.20271" originrpy="0 0 1.5708" />
     <xacro:arm_joint prefix="bottom_wrist" parent="bicep" child="bottom_wrist" originxyz="0.0 -0.05194 0.269" originrpy="0 0 0" />
